File: z80busCard.kicad_pcb (KiCad board)
At the start: 2 copper layers, 115.6 x 78.1 mm, 18 parts, among them J1 Conn_02x20_Odd_Even, J2 Conn_02x20_Odd_Even, J3 Conn_02x20_Odd_Even, J4 Conn_02x20_Odd_Even, J5 USB_C_Receptacle_PowerOnly_6P, SW1 SW_Push

Commit message: Added schmitt trigger on ~RESET
Also added a ~RESET input connector.
Parts:
- added C2: 0.1u, Capacitor_SMD:C_0805_2012Metric_Pad1.18x1.45mm_HandSolder, B.Cu at (113.3, 132.7)
- added J6: Conn_01x04_Pin, Connector_PinHeader_2.54mm:PinHeader_1x04_P2.54mm_Vertical, F.Cu at (86.6, 128.9)
- added U1: 74HC14, Package_DIP:DIP-14_W7.62mm_Socket, F.Cu at (110.9, 137.2)
- renumbered +5V to H1, GND to H2
Connections:
- C1 pad 1: /~{RESET} -> /~{RESET_INPUT}
- J5 pad SH: GND -> (no net)
- R1 pad 2: /~{RESET} -> /~{RESET_INPUT}
- SW1 pad 2: /~{RESET} -> /~{RESET_INPUT}
Routing:
- net /~{RESET_INPUT}: track 0.00 -> 80.5 mm
- net /~{RESET}: track 112.2 -> 118.6 mm
- net +5V: track 79.3 -> 83.0 mm
- net Net-(U1-Pad2): track 0.00 -> 2.54 mm
Other:
- board text added: "Z80 bus card v1.4 2026-07-22"
- board text added: "~{RESET} Input"
- board text removed: "Z80 bus card v1.3 2026-05-17"
