File: z80busCard.kicad_sch (KiCad schematic)
At the start: 14 parts, among them J1 Conn_02x20_Odd_Even, J2 Conn_02x20_Odd_Even, J3 Conn_02x20_Odd_Even, J4 Conn_02x20_Odd_Even, J5 USB_C_Receptacle_PowerOnly_6P, SW1 SW_Push

Commit message: Added schmitt trigger on ~RESET
Also added a ~RESET input connector.
Parts:
- added C2: 0.1u, Capacitor_SMD:C_0805_2012Metric_Pad1.18x1.45mm_HandSolder, symbol Device:C
- added J6: Conn_01x04_Pin, Connector_PinHeader_2.54mm:PinHeader_1x04_P2.54mm_Vertical, symbol Connector:Conn_01x04_Pin
- added U1: 74HC14, Package_DIP:DIP-14_W7.62mm_Socket, symbol 74xx:74HC14
Connections:
- net +5V: now also C2.1, U1.14 (VCC)
- net GND: now also C2.2, U1.11, U1.13, U1.5, U1.7 (GND), U1.9
- net ~{RESET}: now also U1.4; no longer C1.1, R1.2, SW1.2
- new net: U1.2, U1.3
- new net ~{RESET_INPUT}: C1.1, J6.1 (Pin_1), J6.2 (Pin_2), J6.3 (Pin_3), J6.4 (Pin_4), R1.2, SW1.2, U1.1
- no-connect marks 0 -> 4
Other:
- moved on the sheet: D201, J1, J2, J3, J4, J5, R2, R218, R3
